File: rule169/rule169.kicad_pcb (KiCad board)
At the start: 2 copper layers, 112.1 x 87.7 mm, 39 parts, among them U1 xiao-ble

Commit message: add project files
Parts:
- removed the REF** at (280.0, 111.0)
- removed the REF** at (276.1, 96.8)
- removed the REF** at (273.3, 104.6)
- removed the REF** at (269.8, 110.0)
- added ?: , , F.Cu at (32.3, 39.7)
- added ?: , , F.Cu at (259.1, 80.8)
- added ?: , , F.Cu at (287.3, 88.7)
- added ?: , , F.Cu at (33.3, 45.2)
- added ?: , , F.Cu at (219.5, 80.8)
- added ?: , , F.Cu at (31.3, 34.2)
- added ?: , , F.Cu at (247.7, 88.7)
- added L1: LED, Keyboard Footprints:LED_3mm_reversible, F.Cu at (152.3, 45.5)
- added L2: LED, Keyboard Footprints:LED_3mm_reversible, F.Cu at (150.4, 34.5)
- added L3: LED, Keyboard Footprints:LED_3mm_reversible, F.Cu at (151.3, 40.0)
- added R1: 220, Keyboard Footprints:R_1206_DoubleSided, B.Cu at (152.9, 52.4)
- added R2: 220, Keyboard Footprints:R_1206_DoubleSided, B.Cu at (146.8, 52.4)
- added R3: 220, Keyboard Footprints:R_1206_DoubleSided, B.Cu at (149.9, 52.3)
- added REF**: M2 Hole, Keyboard Footprints:M2 Hole, F.Cu at (259.0, 29.2)
- added REF**: M2 Hole, Keyboard Footprints:M2 Hole, F.Cu at (219.4, 29.2)
- added REF**: Battery lipo 601235, Keyboard Footprints:Battery lipo 601235, F.Cu at (243.8, 68.7)
- added RSW1: SW_Push, Keyboard Footprints:ResetSW, F.Cu at (252.0, 55.2)
- U1: footprint Keyboard Footprints:xiao-ble-tht -> Keyboard Footprints:xiao seed ble
- moved D5 105.5 mm to (248.7, 64.6), turned to -90 degrees
- moved D9 105.1 mm to (248.7, 74.0), turned to -90 degrees
- moved D1 84.7 mm to (248.7, 54.9), turned to -90 degrees
- moved D10 82.7 mm to (245.6, 74.0), turned to -90 degrees
- moved PSW1 82.6 mm to (230.4, 27.0), turned to -90 degrees
- moved D6 81.7 mm to (245.6, 64.6), turned to -90 degrees
- moved D16 66.6 mm to (242.5, 83.4), turned to -90 degrees
- moved D11 62.5 mm to (242.6, 74.0), turned to -90 degrees
- moved D14 62.4 mm to (248.7, 83.4), turned to -90 degrees
- moved D15 61.6 mm to (245.6, 83.4), turned to -90 degrees
- moved D2 60.2 mm to (245.6, 54.9), turned to -90 degrees
- moved D7 59.2 mm to (242.6, 64.6), turned to -90 degrees
- moved D8 55.0 mm to (239.5, 64.6), turned to -90 degrees
- moved U1 54.9 mm to (244.0, 38.4), turned to -90 degrees
- moved D3 54.0 mm to (242.6, 54.9), turned to -90 degrees
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Connections:
- PSW1 pad 1: unconnected-(PSW1-Pad1) -> MCU+
- U1 pad 1: unconnected-(U1-Pad1) -> LED0
- U1 pad 17: unconnected-(U1-Pad17) -> RESET
- U1 pad 2: unconnected-(U1-Pad2) -> LED1
- U1 pad 20: MCU- -> GND
- U1 pad 3: unconnected-(U1-Pad3) -> LED2
Routing:
- net col3: track 0.00 -> 453.3 mm
- net col2: track 0.00 -> 355.2 mm
- net col1: track 0.00 -> 334.7 mm
- net col0: track 0.00 -> 197.6 mm
- net Net-(D5-Pad2): track 0.00 -> 140.8 mm
- net Net-(D9-Pad2): track 0.00 -> 126.5 mm
- net Net-(D1-Pad2): track 0.00 -> 123.8 mm
- net Net-(D6-Pad2): track 0.00 -> 115.2 mm
- net Net-(D10-Pad2): track 0.00 -> 104.0 mm
- net Net-(D2-Pad2): track 0.00 -> 101.0 mm
- net Net-(D7-Pad2): track 0.00 -> 94.7 mm
- net Net-(D16-Pad2): track 0.00 -> 87.8 mm
- net Net-(D11-Pad2): track 0.00 -> 87.0 mm
- net Net-(D13-Pad2): track 0.00 -> 77.8 mm
- net Net-(D3-Pad2): track 0.00 -> 77.3 mm
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- added copper zone on B.Cu, net GND
- added copper zone on F.Cu, net GND
Other:
- board size 112.1 x 87.7 mm -> 276.9 x 90.4 mm
